Commit message: sync collision with visual

File: linorobot2_description/urdf/sensors/laser.urdf.xacro (robot description, xacro)
@@ -13,5 +13,5 @@
       </visual>
       <collision>
-        <origin xyz="0 0 0" rpy="${pi/2} 0 0"/>
+        <origin xyz="0 0 -0.025" rpy="0 0 0"/>
         <geometry>
           <cylinder radius="0.0375" length="0.05"/>
