Commit message: added meshes

File: linorobot2_description/urdf/mech/base.urdf.xacro (robot description, xacro)
@@ -1,5 +1,5 @@
 <?xml version="1.0"?>
 <robot xmlns:xacro="http://ros.org/wiki/xacro">
-  <xacro:macro name="base" params="length width height mass wheel_radius wheel_pos_z">
+  <xacro:macro name="base" params="length width height mass wheel_radius wheel_pos_z mesh scale">
     <link name="base_footprint"/>
     <link name="base_link">
@@ -7,13 +7,10 @@
         <origin xyz="0 0 0" rpy="0 0 0"/>
         <geometry>
-          <box size="${length} ${width} ${height}"/>
-          <!-- <mesh filename="" scale="0.001 0.001 0.001"/> -->
+          <!-- <box size="${length} ${width} ${height}"/> -->
+          <mesh filename="${mesh}" scale="${scale} ${scale} ${scale}"/>
         </geometry>
-        <material name="yellow">
-          <color rgba="0.8784 0.6627 0.6627 1.0"/>
-        </material>
       </visual>
       <collision>
-        <origin xyz="0 0 0" rpy="0 0 0"/>
+        <origin xyz="0 0 ${height/2}" rpy="0 0 0"/>
         <geometry>
           <box size="${length} ${width} ${height}"/>
@@ -29,12 +26,5 @@
     </link>
     <gazebo reference="base_link">
-      <visual>
-        <material>
-          <ambient>0.8392 0.6314 0.0 1.0</ambient>
-          <diffuse>0.8392 0.6314 0.0 1.0</diffuse>
-          <specular>0.99 0.99 0.99 1.0</specular>
-          <emissive>0.0 0.0 0.0 0.0</emissive>
-        </material>
-      </visual>
+      <material>Gazebo/FlatBlack</material>
     </gazebo>
     <joint name="base_to_footprint" type="fixed">

File: linorobot2_description/urdf/mech/caster_wheel.urdf.xacro (robot description, xacro)
@@ -36,4 +36,5 @@
         <mu1>0.01</mu1>
         <mu2>0.01</mu2>
+        <material>Gazebo/FlatBlack</material>
     </gazebo>
     <joint name="${side}_caster_wheel_joint" type="fixed">

File: linorobot2_description/urdf/mech/wheel.urdf.xacro (robot description, xacro)
@@ -1,10 +1,34 @@
 <?xml version="1.0"?>
 <robot xmlns:xacro="http://ros.org/wiki/xacro">
-  <xacro:macro name="wheel" params="side radius width pos_x pos_y pos_z mass">
-    <link name="${side}_wheel_link">
+  <xacro:macro name="wheel" params="side radius width pos_x pos_y pos_z mass rim_mesh wheel_mesh scale">
+    <link name="${side}_rim_link">
       <visual>
+        <origin xyz="0 0 0" rpy="0 0 0"/>
+        <geometry>
+          <mesh filename="${rim_mesh}" scale="${scale} ${scale} ${scale}"/>
+        </geometry>
+        <material name="blue">
+            <color rgba="0.1764 0.4588 0.8509 1.0"/>
+        </material>
+      </visual>
+      <collision>
         <origin xyz="0 0 0" rpy="${pi/2} 0 0"/>
         <geometry>
           <cylinder radius="${radius}" length="${width}"/>
+        </geometry>
+      </collision>
+      <inertial>
+        <origin xyz="0 0 0" rpy="0 0 0"/>
+        <mass value="${mass}"/>
+        <inertia ixx="${(2/5) * mass * (radius * radius)}" ixy="0" ixz="0"
+                 iyy="${(2/5) * mass * (radius * radius)}" iyz="0"
+                 izz="${(2/5) * mass * (radius * radius)}" />
+      </inertial>
+    </link>
+    <link name="${side}_wheel_link">
+      <visual>
+        <origin xyz="0 0 0" rpy="0 0 0"/>
+        <geometry>
+          <mesh filename="${wheel_mesh}" scale="${scale} ${scale} ${scale}"/>
         </geometry>
         <material name="blue">
@@ -27,12 +51,8 @@
     </link>
     <gazebo reference="${side}_wheel_link">
-      <visual>
-        <material>
-          <ambient>0.1764 0.4588 0.8509 1.0</ambient>
-          <diffuse>0.1764 0.4588 0.8509 1.0</diffuse>
-          <specular>0.1764 0.4588 0.8509 1.0</specular>
-          <emissive>0.0 0.0 0.0 0.0</emissive>
-        </material>
-      </visual>
+      <material>Gazebo/FlatBlack</material>
+    </gazebo>
+    <gazebo reference="${side}_rim_link">
+      <material>Gazebo/White</material>
     </gazebo>
     <joint name="${side}_wheel_joint" type="continuous">
@@ -42,4 +62,10 @@
       <origin xyz="${pos_x} ${pos_y} ${pos_z}" rpy="0 0 0"/>
     </joint>
+    <joint name="${side}_rim_joint" type="fixed">
+      <axis xyz="0 1 0" />
+      <parent link="${side}_wheel_link"/>
+      <child link="${side}_rim_link"/>
+      <origin xyz="0 0 0" rpy="0 0 0"/>
+    </joint>
   </xacro:macro>
 </robot>

File: linorobot2_description/urdf/robots/square.urdf.xacro (robot description, xacro)
@@ -3,5 +3,5 @@
   <xacro:property name="base_length" value="0.25" />
   <xacro:property name="base_width" value="0.25" />
-  <xacro:property name="base_height" value="0.003" />
+  <xacro:property name="base_height" value="0.358" />
   <xacro:property name="base_mass" value="1" />
   <xacro:property name="wheel_radius" value="0.045" />
@@ -9,5 +9,5 @@
   <xacro:property name="wheel_pos_x" value="0.08" />
   <xacro:property name="wheel_pos_y" value="0.12" />
-  <xacro:property name="wheel_pos_z" value="-0.045" />
+  <xacro:property name="wheel_pos_z" value="-0.04" />
   <xacro:property name="wheel_mass" value=".1" />
   <xacro:property name="wheel_torque" value="20" />
@@ -37,4 +37,6 @@
     wheel_radius="${wheel_radius}"
     wheel_pos_z="${wheel_pos_z}"
+    mesh="$(find linorobot2_description)/urdf/mesh/base.stl"
+    scale="0.001"
   />
   <xacro:wheel
@@ -46,4 +48,7 @@
     pos_z="${wheel_pos_z}"
     mass="${wheel_mass}"
+    rim_mesh="$(find linorobot2_description)/urdf/mesh/rim.stl"
+    wheel_mesh="$(find linorobot2_description)/urdf/mesh/wheel.stl"
+    scale="0.001"
   />
   <xacro:wheel
@@ -55,4 +60,7 @@
     pos_z="${wheel_pos_z}"
     mass="${wheel_mass}"
+    rim_mesh="$(find linorobot2_description)/urdf/mesh/rim.stl"
+    wheel_mesh="$(find linorobot2_description)/urdf/mesh/wheel.stl"
+    scale="0.001"
   />
   <xacro:if value="${front_caster_wheel}">

Commit message: added color

File: linorobot2_description/urdf/mech/base.urdf.xacro (robot description, xacro)
@@ -2,4 +2,10 @@
 <robot xmlns:xacro="http://ros.org/wiki/xacro">
   <xacro:macro name="base" params="length width height mass wheel_radius wheel_pos_z mesh scale">
+    <material name="black">
+      <color rgba="0.15 0.15 0.15 1.0"/>
+    </material>
+    <material name="white">
+      <color rgba="0.9 0.9 0.9 1.0"/>
+    </material>
     <link name="base_footprint"/>
     <link name="base_link">
@@ -10,4 +16,5 @@
           <mesh filename="${mesh}" scale="${scale} ${scale} ${scale}"/>
         </geometry>
+        <material name="black"/>
       </visual>
       <collision>

File: linorobot2_description/urdf/mech/wheel.urdf.xacro (robot description, xacro)
@@ -8,7 +8,5 @@
           <mesh filename="${rim_mesh}" scale="${scale} ${scale} ${scale}"/>
         </geometry>
-        <material name="blue">
-            <color rgba="0.1764 0.4588 0.8509 1.0"/>
-        </material>
+        <material name="white"/>
       </visual>
       <collision>
@@ -32,7 +30,5 @@
           <mesh filename="${wheel_mesh}" scale="${scale} ${scale} ${scale}"/>
         </geometry>
-        <material name="blue">
-            <color rgba="0.1764 0.4588 0.8509 1.0"/>
-        </material>
+        <material name="black"/>
       </visual>
       <collision>

File: linorobot2_description/urdf/robots/square.urdf.xacro (robot description, xacro)
@@ -37,5 +37,5 @@
     wheel_radius="${wheel_radius}"
     wheel_pos_z="${wheel_pos_z}"
-    mesh="$(find linorobot2_description)/urdf/mesh/base.stl"
+    mesh="file://$(find linorobot2_description)/urdf/mesh/base.stl"
     scale="0.001"
   />
@@ -48,6 +48,6 @@
     pos_z="${wheel_pos_z}"
     mass="${wheel_mass}"
-    rim_mesh="$(find linorobot2_description)/urdf/mesh/rim.stl"
-    wheel_mesh="$(find linorobot2_description)/urdf/mesh/wheel.stl"
+    rim_mesh="file://$(find linorobot2_description)/urdf/mesh/rim.stl"
+    wheel_mesh="file://$(find linorobot2_description)/urdf/mesh/wheel.stl"
     scale="0.001"
   />
@@ -60,6 +60,6 @@
     pos_z="${wheel_pos_z}"
     mass="${wheel_mass}"
-    rim_mesh="$(find linorobot2_description)/urdf/mesh/rim.stl"
-    wheel_mesh="$(find linorobot2_description)/urdf/mesh/wheel.stl"
+    rim_mesh="file://$(find linorobot2_description)/urdf/mesh/rim.stl"
+    wheel_mesh="file://$(find linorobot2_description)/urdf/mesh/wheel.stl"
     scale="0.001"
   />

Commit message: used mesh for collision to prevent blocking of laser

File: linorobot2_description/urdf/mech/base.urdf.xacro (robot description, xacro)
@@ -21,5 +21,5 @@
         <origin xyz="0 0 ${height/2}" rpy="0 0 0"/>
         <geometry>
-          <box size="${length} ${width} ${height}"/>
+          <mesh filename="${mesh}" scale="${scale} ${scale} ${scale}"/>
         </geometry>
       </collision>

Commit message: sync collision mesh with visual mesh

File: linorobot2_description/urdf/mech/base.urdf.xacro (robot description, xacro)
@@ -19,5 +19,5 @@
       </visual>
       <collision>
-        <origin xyz="0 0 ${height/2}" rpy="0 0 0"/>
+        <origin xyz="0 0 0" rpy="0 0 0"/>
         <geometry>
           <mesh filename="${mesh}" scale="${scale} ${scale} ${scale}"/>
