Commit message: updated robot arm urdf

File: linorobot2_description/urdf/robots/square_mm.urdf.xacro (robot description, xacro)
@@ -22,5 +22,5 @@
   <xacro:include filename="$(find linorobot2_description)/urdf/sensors/depth_sensor.urdf.xacro" />
   <xacro:include filename="$(find linorobot2_description)/urdf/controllers/diff_drive.urdf.xacro" />
-  <xacro:include filename="$(find robot_arm_description)/urdf/arm_mech.urdf.xacro" />
+  <xacro:include filename="$(find robot_arm_description)/urdf/assembled_arm.urdf.xacro" />
   <xacro:property name="laser_pose">
     <origin xyz="0.0 0 0.325" rpy="-3.1416 0 0"/>
@@ -118,4 +118,7 @@
       </inertial>
   </link>
+  <gazebo reference="base_mount">
+    <material>Gazebo/FlatBlack</material>
+  </gazebo>
   <joint name="base_to_arm" type="fixed">
     <parent link="base_link"/>
@@ -123,4 +126,4 @@
     <origin xyz="0 0 0.363" rpy="0 0 0"/>
   </joint>
-  <xacro:arm_mech parent="base_mount" use_sim_time="$(arg use_sim_time)" />
+  <xacro:assembled_arm parent="base_mount" use_sim_time="$(arg use_sim_time)" />
 </robot>
